Commit message: 测试

File: source/Y1_1Pace/Y1_1Pace/tasks/manager_based/Y1_1_robot/urdf/Y1_1_Link.urdf (robot description, URDF)
Before this commit: robot Y1_1, 2 links, 2 joints
Joints:
- removed joint l_knee_pitch_joint
- joint l_hip_yaw_joint: limit lower=-2.792526803190927 upper=2.792526803190927 effort=36.0 velocity=10.5 -> effort=10.0 velocity=6

Commit message: 改关节

File: source/Y1_1Pace/Y1_1Pace/tasks/manager_based/Y1_1_robot/urdf/Y1_1_Link.urdf (robot description, URDF)
Before this commit: robot Y1_1, 2 links, 1 joints
Joints:
- joint l_hip_yaw_joint: limit effort=10.0 velocity=6 -> lower=-2.792526803190927 upper=2.792526803190927 effort=36.0 velocity=10.5; type continuous -> revolute

Commit message: change back limit

File: source/Y1_1Pace/Y1_1Pace/tasks/manager_based/Y1_1_robot/urdf/Y1_1_Link.urdf (robot description, URDF)
Before this commit: robot Y1_1, 2 links, 1 joints
Joints:
- joint l_hip_yaw_joint: limit effort=10.0 velocity=6 -> lower=-2.792526803190927 upper=2.792526803190927 effort=36.0 velocity=10.5

Commit message: 【修改】urdf改为revolute，其他

File: source/Y1_1Pace/Y1_1Pace/tasks/manager_based/Y1_1_robot/urdf/Y1_1_Link.urdf (robot description, URDF)
Before this commit: robot Y1_1, 2 links, 1 joints
Joints:
- joint l_hip_yaw_joint: type continuous -> revolute

Commit message: 【模型】增加0.5倍的连杆质量，其他参数不变

File: source/Y1_1Pace/Y1_1Pace/tasks/manager_based/Y1_1_robot/urdf/Y1_1_Link.urdf (robot description, URDF)
Before this commit: robot Y1_1, 2 links, 1 joints
Links:
- link l_hip_roll_Link: mass 0.74464439636084 -> 1.0

Commit message: data:change the link mass

File: source/Y1_1Pace/Y1_1Pace/tasks/manager_based/Y1_1_robot/urdf/Y1_1_Link.urdf (robot description, URDF)
Before this commit: robot Y1_1, 2 links, 1 joints
Links:
- link l_hip_yaw_Link: mass 1.0973721550832 -> 1.5
