Commit message: 删除其他urdf配置

File: source/Y1_1Pace/Y1_1Pace/tasks/manager_based/RS06/urdf/single_joint.urdf (robot description, URDF)
Before this commit: robot Y1_1, 18 links, 17 joints
Links:
- removed link l_ankle_pitch_Link
- removed link l_ankle_roll_Link
- removed link l_elbow_pitch_Link
- removed link l_elbow_yaw_Link
- removed link l_hip_pitch_Link
- removed link l_hip_roll_Link
- removed link l_hip_yaw_Link
- removed link l_knee_pitch_Link
- removed link l_shoulder_pitch_Link
- removed link l_shoulder_roll_Link
- removed link l_wrist_pitch_Link
- removed link r_elbow_pitch_Link
- removed link r_elbow_yaw_Link
- removed link r_shoulder_pitch_Link
- removed link r_shoulder_roll_Link
- removed link r_wrist_pitch_Link
- link waist_yaw_Link: mass 1.76450922077218 -> 0.000
Joints:
- removed joint l_ankle_pitch_joint
- removed joint l_ankle_roll_joint
- removed joint l_elbow_pitch_joint
- removed joint l_elbow_yaw_joint
- removed joint l_hip_pitch_joint
- removed joint l_hip_roll_joint
- removed joint l_hip_yaw_joint
- removed joint l_knee_pitch_joint
- removed joint l_shoulder_pitch_joint
- removed joint l_shoulder_roll_joint
- removed joint l_wrist_pitch_joint
- removed joint r_elbow_pitch_joint
- removed joint r_elbow_yaw_joint
- removed joint r_shoulder_pitch_joint
- removed joint r_shoulder_roll_joint
- removed joint r_wrist_pitch_joint
- joint waist_yaw_joint: limit lower=-2.5307274153917776 upper=2.5307274153917776 effort=36.0 velocity=10.5 -> lower=-2.5307274153917776 upper=2.5307274153917776 effort=36.0 velocity=50; type fixed -> revolute

Commit message: 其他参数准备就绪，但测试最高转速保持在额定转速左右，重新提取数据

File: source/Y1_1Pace/Y1_1Pace/tasks/manager_based/RS06/urdf/single_joint.urdf (robot description, URDF)
Before this commit: robot Y1_1, 2 links, 1 joints
Joints:
- joint waist_yaw_joint: limit lower=-2.5307274153917776 upper=2.5307274153917776 effort=36.0 velocity=50 -> lower=-2.5307274153917776 upper=2.5307274153917776 effort=36.0 velocity=10
